Commit message: Match OpenAI CartPole environment
https://github.com/openai/gym/blob/master/gym/envs/classic_control/cartpole.py

File: models/CartPole/CartPole.urdf (robot description, URDF)
Before this commit: robot cartpole_xacro, 4 links, 3 joints
Links:
- link cart: mass 3 -> 1.0
- link pole: mass 1 -> 0.1; geometry visual cylinder length=1.0 radius=0.005
- link rail: geometry visual cylinder length=5 radius=0.005
Joints:
- joint linear: limit lower=-0.9 upper=0.9 effort=500 velocity=10 -> lower=-2.4 upper=2.4 effort=500 velocity=10

File: models/CartPole/CartPole.urdf.xacro (robot description, xacro)
@@ -1,6 +1,8 @@
 <?xml version='1.0' encoding='UTF-8'?>
 <robot name="cartpole_xacro" xmlns:xacro="http://www.ros.org/wiki/xacro">
+  <!-- CartPole properties match the OpenAI Gym CartPole-v1 environment -->
+  <!-- https://github.com/openai/gym/blob/master/gym/envs/classic_control/cartpole.py -->
   <xacro:property name="rail_height" value="0.5" />
-  <xacro:property name="rail_length" value="2" />
+  <xacro:property name="rail_length" value="5" />
   <xacro:property name="rail_radius" value="0.005" />
   <xacro:property name="rail_mass" value="5" />
@@ -8,8 +10,8 @@
   <xacro:property name="cart_size_y" value="0.2" />
   <xacro:property name="cart_size_z" value="0.05" />
-  <xacro:property name="cart_mass" value="3" />
-  <xacro:property name="pole_length" value="0.5" />
+  <xacro:property name="cart_mass" value="1.0" />
+  <xacro:property name="pole_length" value="1.0" />
   <xacro:property name="pole_radius" value="0.005" />
-  <xacro:property name="pole_mass" value="1" />
+  <xacro:property name="pole_mass" value="0.1" />
   <xacro:property name="theta_0" value="0" />
   <xacro:property name="epsilon" value="1e-09"/>
