Commit message: Update Cartpole and Pendulum models
- Converted with a recent sdformat version that does not use parent_model_frame
- Fixed few errors in inertia calculation
- Add right inertial elements also for support links
- Add collision elements

File: gym_ignition_data/CartPole/CartPole.urdf (robot description, URDF)
Before this commit: robot cartpole_xacro, 4 links, 3 joints
Links:
- link cart: geometry collision box size=0.1 0.2 0.05; visual box size=0.1 0.2 0.05
- link pole: geometry collision cylinder length=1.0 radius=0.005; visual cylinder length=1.0 radius=0.005
Joints:
- joint pivot: limit lower=-1.57079632679 upper=1.57079632679 effort=500 velocity=10 -> lower=-6.28318530718 upper=6.28318530718 effort=500 velocity=10; origin xyz=0 0 0.025 rpy=0 0 0 -> xyz=0 0 0.025 rpy=0.0 0 0
- joint world_to_rail: origin xyz=0 0 0.5 rpy=0 0 0 -> xyz=0 0 1.2 rpy=0 0 0

File: gym_ignition_data/CartPole/CartPole.urdf.xacro (robot description, xacro)
@@ -1,151 +1,161 @@
 <?xml version='1.0' encoding='UTF-8'?>
 <robot name="cartpole_xacro" xmlns:xacro="http://www.ros.org/wiki/xacro">
-  <!-- CartPole properties match the OpenAI Gym CartPole-v1 environment -->
-  <!-- https://github.com/openai/gym/blob/master/gym/envs/classic_control/cartpole.py -->
-  <xacro:property name="rail_height" value="0.5" />
-  <xacro:property name="rail_length" value="5" />
-  <xacro:property name="rail_radius" value="0.005" />
-  <xacro:property name="rail_mass" value="5" />
-  <xacro:property name="cart_size_x" value="0.1" />
-  <xacro:property name="cart_size_y" value="0.2" />
-  <xacro:property name="cart_size_z" value="0.05" />
-  <xacro:property name="cart_mass" value="1.0" />
-  <xacro:property name="pole_length" value="1.0" />
-  <xacro:property name="pole_radius" value="0.005" />
-  <xacro:property name="pole_mass" value="0.1" />
-  <xacro:property name="theta_0" value="0" />
-  <xacro:property name="epsilon" value="1e-09"/>
-  <xacro:property name="rgba_black" value="0 0 0 0.8"/>
-  <xacro:property name="rgba_white" value="1 1 1 0.8"/>
-  <xacro:property name="rgba_grey" value="0.2 0.2 0.2 0.8"/>
-  <xacro:property name="rgba_red" value="1 0 0 0.8"/>
-  <xacro:macro name="box_inertia" params="mass dimx dimy dimz xyz rpy">
-    <inertial>
-      <origin xyz="${xyz}" rpy="${rpy}"/>
-      <mass value="${mass}"/>
-      <xacro:property name="ixx" value="${1/12*mass*(dimz*dimz+dimy*dimy)}"/>
-      <xacro:property name="iyy" value="${1/12*mass*(dimx*dimx+dimy*dimy)}"/>
-      <xacro:property name="izz" value="${1/12*mass*(dimx*dimx+dimz*dimz)}"/>
-      <inertia ixx="${ixx}"  ixy="0"  ixz="0" iyy="${iyy}" iyz="0" izz="${izz}" />
-    </inertial>
-  </xacro:macro>
-  <xacro:macro name="cylinder_inertial_element"
-               params="mass rotaxis length radius xyz rpy">
-    <inertial>
-      <origin xyz="${xyz}" rpy="${rpy}"/>
-      <mass value="${mass}"/>
-      <xacro:property name="ixx" value="${1/12*mass*(3*radius*radius+length*length)}"/>
-      <xacro:property name="iyy" value="${1/12*mass*(3*radius*radius+length*length)}"/>
-      <xacro:property name="izz" value="${0.5*mass*radius*radius}"/>
-      <inertia ixx="${ixx}"  ixy="0"  ixz="0" iyy="${iyy}" iyz="0" izz="${izz}" />
-    </inertial>
-  </xacro:macro>
-  <xacro:macro name="mymaterial" params="name rgba">
-    <material name="${name}">
-        <color rgba="${rgba}"/>
+    <!-- CartPole properties match the OpenAI Gym CartPole-v1 environment -->
+    <!-- https://github.com/openai/gym/blob/master/gym/envs/classic_control/cartpole.py -->
+    <xacro:property name="rail_height" value="1.2"/>
+    <xacro:property name="rail_length" value="5"/>
+    <xacro:property name="rail_radius" value="0.005"/>
+    <xacro:property name="rail_mass" value="5"/>
+    <xacro:property name="cart_size_x" value="0.1"/>
+    <xacro:property name="cart_size_y" value="0.2"/>
+    <xacro:property name="cart_size_z" value="0.05"/>
+    <xacro:property name="cart_mass" value="1.0"/>
+    <xacro:property name="pole_length" value="1.0"/>
+    <xacro:property name="pole_radius" value="0.005"/>
+    <xacro:property name="pole_mass" value="0.1"/>
+    <xacro:property name="theta_0" value="0.0"/>
+    <xacro:property name="epsilon" value="1e-09"/>
+    <xacro:property name="rgba_black" value="0 0 0 0.8"/>
+    <xacro:property name="rgba_white" value="1 1 1 0.8"/>
+    <xacro:property name="rgba_grey" value="0.2 0.2 0.2 0.8"/>
+    <xacro:property name="rgba_red" value="1 0 0 0.8"/>
+    <xacro:macro name="box_inertia" params="mass dimx dimy dimz xyz rpy">
+        <inertial>
+            <origin xyz="${xyz}" rpy="${rpy}"/>
+            <mass value="${mass}"/>
+            <xacro:property name="ixx" value="${1/12*mass*(dimy*dimy+dimz*dimz)}"/>
+            <xacro:property name="iyy" value="${1/12*mass*(dimx*dimx+dimz*dimz)}"/>
+            <xacro:property name="izz" value="${1/12*mass*(dimx*dimx+dimy*dimy)}"/>
+            <inertia ixx="${ixx}" ixy="0" ixz="0" iyy="${iyy}" iyz="0" izz="${izz}"/>
+        </inertial>
+    </xacro:macro>
+    <xacro:macro name="cylinder_inertial_element"
+                 params="mass length radius xyz rpy">
+        <inertial>
+            <origin xyz="${xyz}" rpy="${rpy}"/>
+            <mass value="${mass}"/>
+            <xacro:property name="ixx"
+                            value="${1/12*mass*(3*radius*radius+length*length)}"/>
+            <xacro:property name="iyy"
+                            value="${1/12*mass*(3*radius*radius+length*length)}"/>
+            <xacro:property name="izz" value="${0.5*mass*radius*radius}"/>
+            <inertia ixx="${ixx}" ixy="0" ixz="0" iyy="${iyy}" iyz="0" izz="${izz}"/>
+        </inertial>
+    </xacro:macro>
+    <xacro:macro name="mymaterial" params="name rgba">
+        <material name="${name}">
+            <color rgba="${rgba}"/>
+        </material>
+    </xacro:macro>
+    <xacro:macro name="gzmaterial" params="reference rgba">
+        <gazebo reference="${reference}">
+            <visual>
+                <material>
+                    <ambient>${rgba}</ambient>
+                    <diffuse>${rgba}</diffuse>
+                    <specular>${rgba}</specular>
+                    <emissive>${rgba}</emissive>
+                </material>
+            </visual>
+        </gazebo>
+    </xacro:macro>
+    <!-- ====== -->
+    <!-- COLORS -->
+    <!-- ====== -->
+    <material name="black">
+        <color rgba="${rgba_black}"/>
     </material>
-  </xacro:macro>
-  <xacro:macro name="gzmaterial" params="reference rgba">
-    <gazebo reference="${reference}">
-      <visual>
-        <material>
-            <ambient>${rgba}</ambient>
-            <diffuse>${rgba}</diffuse>
-            <specular>${rgba}</specular>
-            <emissive>${rgba}</emissive>
-            <script>
-              <uri></uri>
-              <name></name>
-            </script>
-        </material>
+    <material name="white">
+        <color rgba="${rgba_white}"/>
+    </material>
+    <material name="grey">
+        <color rgba="${rgba_grey}"/>
+    </material>
+    <xacro:gzmaterial reference="rail" rgba="${rgba_black}"/>
+    <xacro:gzmaterial reference="cart" rgba="${rgba_grey}"/>
+    <xacro:gzmaterial reference="pole" rgba="${rgba_red}"/>
+    <!-- ===== -->
+    <!-- LINKS -->
+    <!-- ===== -->
+    <link name="world"/>
+    <link name="rail">
+        <xacro:cylinder_inertial_element mass="${rail_mass}"
+                                         length="${rail_length}"
+                                         radius="${rail_radius}"
+                                         xyz="0 0 0"
+                                         rpy="${pi/2} 0 0"/>
+        <visual>
+            <geometry>
+                <cylinder length="${rail_length}" radius="${rail_radius}"/>
+            </geometry>
+            <origin xyz="0 0 0" rpy="${pi/2} 0 0"/>
+            <xacro:mymaterial name="black" rgba="${rgba_black}"/>
         </visual>
-    </gazebo>
-  </xacro:macro>
-  <!-- ====== -->
-  <!-- COLORS -->
-  <!-- ====== -->
-  <material name="black">
-    <color rgba="${rgba_black}"/>
-  </material>
-  <material name="white">
-    <color rgba="${rgba_white}"/>
-  </material>
-  <material name="grey">
-    <color rgba="${rgba_grey}"/>
-  </material>
-  <xacro:gzmaterial reference="rail" rgba="${rgba_black}"/>
-  <xacro:gzmaterial reference="cart" rgba="${rgba_grey}"/>
-  <xacro:gzmaterial reference="pole" rgba="${rgba_red}"/>
-  <!-- ===== -->
-  <!-- LINKS -->
-  <!-- ===== -->
-  <link name="world"/>
-  <link name="rail">
-    <inertial>
-      <!-- This link is fixed, inertial values are not relevant -->
-      <origin xyz="0 0 0" rpy="0 0 0"/>
-      <mass value="${rail_mass}"/>
-      <inertia ixx="100"  ixy="0"  ixz="0" iyy="100" iyz="0" izz="100" />
-    </inertial>
-    <visual>
-      <geometry>
-        <cylinder length="${rail_length}" radius="${rail_radius}"/>
-      </geometry>
-      <origin xyz="0 0 0" rpy="${pi/2} 0 0"/>
-      <xacro:mymaterial name="black" rgba="${rgba_black}" />
-    </visual>
-  </link>
-  <link name="cart">
-    <xacro:box_inertia mass="${cart_mass}"
-                       dimx="${cart_size_x}"
-                       dimy="${cart_size_y}"
-                       dimz="${cart_size_z}"
-                       xyz="0 0 0"
-                       rpy="0 0 0"/>
-    <visual>
-      <geometry>
-        <box size="${cart_size_x} ${cart_size_y} ${cart_size_z}"/>
-      </geometry>
-      <origin xyz="0 0 0" rpy="0 0 0"/>
-      <xacro:mymaterial name="grey" rgba="${rgba_grey}" />
-    </visual>
-  </link>
-  <link name="pole">
-    <xacro:cylinder_inertial_element mass="${pole_mass}"
-                                     rotaxis="x"
-                                     length="${pole_length}"
-                                     radius="${pole_radius}"
-                                     xyz="0 0 ${pole_length/2}"
-                                     rpy="0 0 0"/>
-    <visual>
-      <geometry>
-        <cylinder length="${pole_length}" radius="${pole_radius}"/>
-      </geometry>
-      <origin xyz="0 0 ${pole_length/2}" rpy="0 0 0"/>
-      <xacro:mymaterial name="red" rgba="${rgba_red}" />
-    </visual>
-  </link>
-  <!-- ====== -->
-  <!-- JOINTS -->
-  <!-- ====== -->
-  <!--  http://gazebosim.org/tutorials/?tut=ros_urdf#RigidlyFixingAModeltotheWorld-->
-  <joint name="world_to_rail" type="fixed">
-    <parent link="world"/>
-    <child link="rail"/>
-    <origin xyz="0 0 ${rail_height}" rpy="0 0 0" />
-  </joint>
-  <joint name="linear" type="prismatic">
-    <parent link="rail" />
-    <child link="cart" />
-    <axis xyz="0 1 0" />
-    <origin xyz="0 0 0" rpy="0 0 0" />
-    <limit lower="-${rail_length/2-cart_size_y/2}" upper="${rail_length/2-cart_size_y/2}" effort="500" velocity="10"/>
-  </joint>
-  <joint name="pivot" type="continuous">
-    <parent link="cart" />
-    <child link="pole" />
-    <axis xyz="1 0 0"/>
-    <origin xyz="0 0 ${cart_size_z/2}" rpy="${theta_0} 0 0" />
-    <limit lower="-${pi/2}" upper="${pi/2}" effort="500" velocity="10"/>
-  </joint>
+    </link>
+    <link name="cart">
+        <xacro:box_inertia mass="${cart_mass}"
+                           dimx="${cart_size_x}"
+                           dimy="${cart_size_y}"
+                           dimz="${cart_size_z}"
+                           xyz="0 0 0"
+                           rpy="0 0 0"/>
+        <visual>
+            <geometry>
+                <box size="${cart_size_x} ${cart_size_y} ${cart_size_z}"/>
+            </geometry>
+            <origin xyz="0 0 0" rpy="0 0 0"/>
+            <xacro:mymaterial name="grey" rgba="${rgba_grey}"/>
+        </visual>
+        <collision>
+            <geometry>
+                <box size="${cart_size_x} ${cart_size_y} ${cart_size_z}"/>
+            </geometry>
+            <origin xyz="0 0 0" rpy="0 0 0"/>
+        </collision>
+    </link>
+    <link name="pole">
+        <xacro:cylinder_inertial_element mass="${pole_mass}"
+                                         length="${pole_length}"
+                                         radius="${pole_radius}"
+                                         xyz="0 0 ${pole_length/2}"
+                                         rpy="0 0 0"/>
+        <visual>
+            <geometry>
+                <cylinder length="${pole_length}" radius="${pole_radius}"/>
+            </geometry>
+            <origin xyz="0 0 ${pole_length/2}" rpy="0 0 0"/>
+            <xacro:mymaterial name="red" rgba="${rgba_red}"/>
+        </visual>
+        <collision>
+            <geometry>
+                <cylinder length="${pole_length}" radius="${pole_radius}"/>
+            </geometry>
+            <origin xyz="0 0 ${pole_length/2}" rpy="0 0 0"/>
+            <xacro:mymaterial name="red" rgba="${rgba_red}"/>
+        </collision>
+    </link>
+    <!-- ====== -->
+    <!-- JOINTS -->
+    <!-- ====== -->
+    <!-- http://gazebosim.org/tutorials/?tut=ros_urdf#RigidlyFixingAModeltotheWorld -->
+    <joint name="world_to_rail" type="fixed">
+        <parent link="world"/>
+        <child link="rail"/>
+        <origin xyz="0 0 ${rail_height}" rpy="0 0 0"/>
+    </joint>
+    <joint name="linear" type="prismatic">
+        <parent link="rail"/>
+        <child link="cart"/>
+        <axis xyz="0 1 0"/>
+        <origin xyz="0 0 0" rpy="0 0 0"/>
+        <limit lower="-${rail_length/2-cart_size_y/2}"
+               upper="${rail_length/2-cart_size_y/2}" effort="500" velocity="10"/>
+    </joint>
+    <joint name="pivot" type="continuous">
+        <parent link="cart"/>
+        <child link="pole"/>
+        <axis xyz="1 0 0"/>
+        <origin xyz="0 0 ${cart_size_z/2}" rpy="${theta_0} 0 0"/>
+        <limit lower="-${2*pi}" upper="${2*pi}" effort="500" velocity="10"/>
+    </joint>
 </robot>

File: gym_ignition_data/Pendulum/Pendulum.urdf (robot description, URDF)
Before this commit: robot pendulum_xacro, 3 links, 2 joints
Links:
- removed link world
- link pendulum: geometry collision cylinder length=0.5 radius=0.01; visual cylinder length=0.02 radius=0.03
- link support: mass 10 -> 1000; geometry collision box size=0.05 0.1 0.6; visual box size=0.05 0.1 0.6
Joints:
- removed joint world_to_support
- joint pivot: origin xyz=0.035 0 -0.03 rpy=0.0 0 0 -> xyz=0.035 0 0.57 rpy=0.0 0 0

File: gym_ignition_data/Pendulum/Pendulum.urdf.xacro (robot description, xacro)
@@ -9,5 +9,5 @@
     <xacro:property name="support_y" value="0.1"/>
     <xacro:property name="support_z" value="${pendulum_length*1.2}"/>
-    <xacro:property name="support_mass" value="10"/>
+    <xacro:property name="support_mass" value="1000"/>
     <xacro:property name="rgba_black" value="0 0 0 0.8"/>
     <xacro:property name="rgba_white" value="1 1 1 0.8"/>
@@ -15,5 +15,5 @@
     <xacro:property name="rgba_red" value="1 0 0 0.8"/>
     <xacro:macro name="cylinder_inertial_element"
-                 params="mass rotaxis length radius xyz rpy">
+                 params="mass length radius xyz rpy">
         <inertial>
             <origin xyz="${xyz}" rpy="${rpy}"/>
@@ -24,4 +24,18 @@
                             value="${1/12*mass*(3*radius*radius+length*length)}"/>
             <xacro:property name="izz" value="${0.5*mass*radius*radius}"/>
+            <inertia ixx="${ixx}" ixy="0" ixz="0" iyy="${iyy}" iyz="0" izz="${izz}"/>
+        </inertial>
+    </xacro:macro>
+    <xacro:macro name="box_inertial_element"
+                 params="mass dimx dimy dimz xyz rpy">
+        <inertial>
+            <origin xyz="${xyz}" rpy="${rpy}"/>
+            <mass value="${mass}"/>
+            <xacro:property name="ixx"
+                            value="${1/12*mass*(dimy*dimy+dimz*dimz)}"/>
+            <xacro:property name="iyy"
+                            value="${1/12*mass*(dimx*dimx+dimz*dimz)}"/>
+            <xacro:property name="izz"
+                            value="${1/12*mass*(dimx*dimx+dimy*dimy)}"/>
             <inertia ixx="${ixx}" ixy="0" ixz="0" iyy="${iyy}" iyz="0" izz="${izz}"/>
         </inertial>
@@ -40,8 +54,4 @@
                     <specular>${rgba}</specular>
                     <emissive>${rgba}</emissive>
-                    <script>
-                        <uri></uri>
-                        <name></name>
-                    </script>
                 </material>
             </visual>
@@ -56,23 +66,27 @@
     <!-- LINKS -->
     <!-- ===== -->
-    <link name="world"/>
     <link name="support">
-        <inertial>
-            <!-- This link is fixed, inertial values are not relevant -->
-            <origin xyz="0 0 ${support_z*0.5}" rpy="0 0 0"/>
-            <mass value="${support_mass}"/>
-            <inertia ixx="1" ixy="0" ixz="0" iyy="1" iyz="0" izz="1"/>
-        </inertial>
+        <xacro:box_inertial_element mass="${support_mass}"
+                                    dimx="${support_x}"
+                                    dimy="${support_y}"
+                                    dimz="${support_z}"
+                                    xyz="0 0 ${support_z*0.5}"
+                                    rpy="0 0 0"/>
         <visual>
             <geometry>
                 <box size="${support_x} ${support_y} ${support_z}"/>
             </geometry>
-            <origin xyz="0 0 -${support_z*0.5}" rpy="0 0 0"/>
+            <origin xyz="0 0 ${support_z*0.5}" rpy="0 0 0"/>
             <xacro:mymaterial name="black" rgba="${rgba_grey}"/>
         </visual>
+        <collision>
+            <geometry>
+                <box size="${support_x} ${support_y} ${support_z}"/>
+            </geometry>
+            <origin xyz="0 0 ${support_z*0.5}" rpy="0 0 0"/>
+        </collision>
     </link>
     <link name="pendulum">
         <xacro:cylinder_inertial_element mass="${pendulum_mass}"
-                                         rotaxis="x"
                                          length="${pendulum_length}"
                                          radius="${pendulum_radius}"
@@ -94,19 +108,19 @@
             <xacro:mymaterial name="red" rgba="${rgba_red}"/>
         </visual>
+        <collision>
+            <geometry>
+                <cylinder length="${pendulum_length}" radius="${pendulum_radius}"/>
+            </geometry>
+            <origin xyz="0 0 ${pendulum_length/2}" rpy="0 0 0"/>
+        </collision>
     </link>
     <!-- ====== -->
     <!-- JOINTS -->
     <!-- ====== -->
-    <!--  http://gazebosim.org/tutorials/?tut=ros_urdf#RigidlyFixingAModeltotheWorld-->
-    <joint name="world_to_support" type="fixed">
-        <parent link="world"/>
-        <child link="support"/>
-        <origin xyz="0 0 ${support_z}" rpy="0 0 0"/>
-    </joint>
     <joint name="pivot" type="continuous">
         <parent link="support"/>
         <child link="pendulum"/>
         <axis xyz="1 0 0"/>
-        <origin xyz="${support_x/2+pendulum_radius} 0 ${-pendulum_circle_radius}"
+        <origin xyz="${support_x/2+pendulum_radius} 0 ${support_z-pendulum_circle_radius}"
                 rpy="${theta_0} 0 0"/>
         <limit lower="${-2*pi}" upper="${2*pi}" effort="500" velocity="10"/>
